Commit message: fixed previous urdf corruption

File: src/OfficeEnv/urdf/my_robot.urdf.xacro (robot description, xacro)
@@ -237,5 +237,5 @@
     </gazebo>
     <joint name="laser_joint" type="fixed">
-        <parent link="chassis"/>
+        <parent link="base_link"/>
         <child link="laser_frame"/>
         <origin xyz="0.122 0 0.212" rpy="0 0 0"/>
@@ -246,5 +246,5 @@
                 <cylinder radius="0.05" length="0.04"/>
             </geometry>
-            <material name="black"/>
+            <material name="grey"/>
         </visual>
         <visual>
@@ -253,5 +253,5 @@
                 <cylinder radius="0.01" length="0.1"/>
             </geometry>
-            <material name="black"/>
+            <material name="grey"/>
         </visual>
         <collision>
@@ -260,10 +260,9 @@
             </geometry>
         </collision>
-        <xacro:inertial_cylinder mass="0.1" length="0.04" radius="0.05">
-            <origin xyz="0 0 0" rpy="0 0 0"/>
-        </xacro:inertial_cylinder>
+        <xacro:cylinder_inertia m="0.1" r="0.05" h="0.04"
+                                    xyz="0 0 0" rpy="0 0 0" />
     </link>
     <gazebo reference="laser_frame">
-        <material>Gazebo/Black</material>
+        <material>Gazebo/grey</material>
         <sensor name="laser" type="ray">
             <pose> 0 0 0 0 0 0 </pose>

Commit message: updated urdf file

File: src/OfficeEnv/urdf/my_robot.urdf.xacro (robot description, xacro)
@@ -169,7 +169,7 @@
             <plugin name="camera_plugin" filename="libgazebo_ros_camera.so">
                 <alwaysOn>true</alwaysOn>
-                <cameraName>camera1</cameraName>
-                <imageTopicName>image_raw</imageTopicName>
-                <cameraInfoTopicName>camera_info</cameraInfoTopicName>
+                <!-- <cameraName>camera1</cameraName> -->
+                <!-- <imageTopicName>image_raw</imageTopicName>
+                <cameraInfoTopicName>camera_info</cameraInfoTopicName> -->
                 <frame_name>camera_link_optical</frame_name>
                 <ros>
@@ -184,7 +184,11 @@
                 <alwaysOn>true</alwaysOn>
                 <updateRate>0.0</updateRate>
+                <cameraName>depth_camera_ir</cameraName>
+                <imageTopicName>/depth_camera/color/image_raw</imageTopicName>
+                <cameraInfoTopicName>/depth_camera/color/camera_info</cameraInfoTopicName>
                 <depthImageTopicName>/depth_camera/depth/image_raw</depthImageTopicName>
                 <depthImageInfoTopicName>/depth_camera/depth/camera_info</depthImageInfoTopicName>
                 <pointCloudTopicName>/depth_camera/depth/points</pointCloudTopicName>
+                <!-- <frameName>camera_link_optical</frameName> -->
                 <pointCloudCutoff>0.5</pointCloudCutoff>
                 <pointCloudCutoffMax>3.0</pointCloudCutoffMax>
@@ -199,4 +203,7 @@
                 <focalLength>0</focalLength>
                 <hackBaseline>0</hackBaseline>
+                <frame_name>camera_link_optical</frame_name>
+                <min_depth>0.1</min_depth>
+                <max_depth>100.0</max_depth>
             </plugin>
         </sensor>
@@ -235,58 +242,3 @@
         </plugin>
     </gazebo>
-    <joint name="laser_joint" type="fixed">
-        <parent link="base_link"/>
-        <child link="laser_frame"/>
-        <origin xyz="0.122 0 0.212" rpy="0 0 0"/>
-    </joint>
-    <link name="laser_frame">
-        <visual>
-            <geometry>
-                <cylinder radius="0.05" length="0.04"/>
-            </geometry>
-            <material name="grey"/>
-        </visual>
-        <visual>
-            <origin xyz="0 0 -0.05"/>
-            <geometry>
-                <cylinder radius="0.01" length="0.1"/>
-            </geometry>
-            <material name="grey"/>
-        </visual>
-        <collision>
-            <geometry>
-                <cylinder radius="0.05" length="0.04"/>
-            </geometry>
-        </collision>
-        <xacro:cylinder_inertia m="0.1" r="0.05" h="0.04"
-                                    xyz="0 0 0" rpy="0 0 0" />
-    </link>
-    <gazebo reference="laser_frame">
-        <material>Gazebo/grey</material>
-        <sensor name="laser" type="ray">
-            <pose> 0 0 0 0 0 0 </pose>
-            <visualize>true</visualize>
-            <update_rate>10</update_rate>
-            <ray>
-                <scan>
-                    <horizontal>
-                        <samples>360</samples>
-                        <min_angle>-3.14</min_angle>
-                        <max_angle>3.14</max_angle>
-                    </horizontal>
-                </scan>
-                <range>
-                    <min>0.3</min>
-                    <max>12</max>
-                </range>
-            </ray>
-            <plugin name="laser_controller" filename="libgazebo_ros_ray_sensor.so">
-                <ros>
-                    <argument>~/out:=scan</argument>
-                </ros>
-                <output_type>sensor_msgs/LaserScan</output_type>
-                <frame_name>laser_frame</frame_name>
-            </plugin>
-        </sensor>
-    </gazebo>
 </robot>

Commit message: Multiple bots depth launch working

File: src/OfficeEnv/urdf/my_robot.urdf.xacro (robot description, xacro)
@@ -1,4 +1,6 @@
 <?xml version="1.0"?>
 <robot name="my_robot"  xmlns:xacro="http://www.ros.org/wiki/xacro">
+    <!-- Prefix for the robot's links and joints -->
+    <xacro:property name="robot_prefix" value="$(arg robot_name)"/>
     <xacro:property name="base_length" value="0.6" />
     <xacro:property name="base_width" value="0.4" />
@@ -39,6 +41,6 @@
         </inertial>
     </xacro:macro>
-    <link name="base_footprint" />
-    <link name="base_link">
+    <link name="${robot_prefix}/base_footprint" />
+    <link name="${robot_prefix}/base_link">
         <visual>
             <geometry>
@@ -57,5 +59,5 @@
                            xyz="0 0 ${base_height / 2.0}" rpy="0 0 0" />
     </link>
-    <link name="right_wheel_link">
+    <link name="${robot_prefix}/right_wheel_link">
         <visual>
             <geometry>
@@ -74,5 +76,5 @@
                                     xyz="0 0 0" rpy="${pi / 2.0} 0 0" />
     </link>
-    <link name="left_wheel_link">
+    <link name="${robot_prefix}/left_wheel_link">
         <visual>
             <geometry>
@@ -91,5 +93,5 @@
                                     xyz="0 0 0" rpy="${pi / 2.0} 0 0" />
     </link>
-    <link name="caster_wheel_link">
+    <link name="${robot_prefix}/caster_wheel_link">
         <visual>
             <geometry>
@@ -108,32 +110,32 @@
                               xyz="0 0 0" rpy="0 0 0" />
     </link>
-    <joint name="base_joint" type="fixed">
-        <parent link="base_footprint" />
-        <child link="base_link" />
+    <joint name="${robot_prefix}/base_joint" type="fixed">
+        <parent link="${robot_prefix}/base_footprint" />
+        <child link="${robot_prefix}/base_link" />
         <origin xyz="0 0 0.1" rpy="0 0 0"/>
     </joint>
-    <joint name="base_right_wheel_joint" type="continuous">
-        <parent link="base_link" />
-        <child link="right_wheel_link" />
+    <joint name="${robot_prefix}/base_right_wheel_joint" type="continuous">
+        <parent link="${robot_prefix}/base_link" />
+        <child link="${robot_prefix}/right_wheel_link" />
         <origin xyz="-0.15 -0.225 0" rpy="0 0 0" />
         <axis xyz="0 1 0" />
     </joint>
-    <joint name="base_left_wheel_joint" type="continuous">
-        <parent link="base_link" />
-        <child link="left_wheel_link" />
+    <joint name="${robot_prefix}/base_left_wheel_joint" type="continuous">
+        <parent link="${robot_prefix}/base_link" />
+        <child link="${robot_prefix}/left_wheel_link" />
         <origin xyz="-0.15 0.225 0" rpy="0 0 0" />
         <axis xyz="0 1 0" />
     </joint>
-    <joint name="base_caster_wheel_joint" type="fixed">
-        <parent link="base_link" />
-        <child link="caster_wheel_link" />
+    <joint name="${robot_prefix}/base_caster_wheel_joint" type="fixed">
+        <parent link="${robot_prefix}/base_link" />
+        <child link="${robot_prefix}/caster_wheel_link" />
         <origin xyz="0.2 0 -0.05" rpy="0 0 0" />
     </joint>
-    <joint name="camera_joint" type="fixed">
-        <parent link="base_link"/>
-        <child link="camera_link"/>
+    <joint name="${robot_prefix}/camera_joint" type="fixed">
+        <parent link="${robot_prefix}/base_link"/>
+        <child link="${robot_prefix}/camera_link"/>
         <origin xyz="0.31 0 0.1" rpy="0 0 0"/>
     </joint>
-    <link name="camera_link">
+    <link name="${robot_prefix}/camera_link">
         <visual>
             <geometry>
@@ -143,11 +145,11 @@
         </visual>
     </link>
-    <joint name="camera_optical_joint" type="fixed">
-        <parent link="camera_link"/>
-        <child link="camera_link_optical"/>
+    <joint name="${robot_prefix}/camera_optical_joint" type="fixed">
+        <parent link="${robot_prefix}/camera_link"/>
+        <child link="${robot_prefix}/camera_link_optical"/>
         <origin xyz="0 0 0" rpy="${-pi/2} 0 ${-pi/2}"/>
     </joint>
-    <link name="camera_link_optical"></link>
-    <gazebo reference="camera_link">
+    <link name="${robot_prefix}/camera_link_optical"></link>
+    <gazebo reference="${robot_prefix}/camera_link">
         <material>Gazebo/Red</material>
         <sensor name="camera" type="depth">
@@ -169,14 +171,5 @@
             <plugin name="camera_plugin" filename="libgazebo_ros_camera.so">
                 <alwaysOn>true</alwaysOn>
-                <!-- <cameraName>camera1</cameraName> -->
-                <!-- <imageTopicName>image_raw</imageTopicName>
-                <cameraInfoTopicName>camera_info</cameraInfoTopicName> -->
-                <frame_name>camera_link_optical</frame_name>
-                <ros>
-                    <argument>/camera/image_raw:=/camera/rgb/image_color</argument>
-                    <argument>/camera/camera_info:=/camera/rgb/camera_info</argument>
-                    <argument>/camera/depth/image_raw:=/camera/depth/image</argument>
-                    <argument>/camera/depth/camera_info:=camera_ab/depth/camera_info</argument>
-                </ros>
+                <frame_name>${robot_prefix}/camera_link_optical</frame_name>
                 <min_depth>0.1</min_depth>
                 <max_depth>100.0</max_depth>
@@ -185,5 +178,4 @@
                 <updateRate>0.0</updateRate>
                 <cameraName>depth_camera_ir</cameraName>
-                <!-- <frameName>camera_link_optical</frameName> -->
                 <pointCloudCutoff>0.5</pointCloudCutoff>
                 <pointCloudCutoffMax>3.0</pointCloudCutoffMax>
@@ -198,20 +190,17 @@
                 <focalLength>0</focalLength>
                 <hackBaseline>0</hackBaseline>
-                <frame_name>camera_link_optical</frame_name>
-                <min_depth>0.1</min_depth>
-                <max_depth>100.0</max_depth>
             </plugin>
         </sensor>
     </gazebo>
-    <gazebo reference="base_link">
+    <gazebo reference="${robot_prefix}/base_link">
         <material>Gazebo/Blue</material>
     </gazebo>
-    <gazebo reference="right_wheel_link">
+    <gazebo reference="${robot_prefix}/right_wheel_link">
         <material>Gazebo/Grey</material>
     </gazebo>
-    <gazebo reference="left_wheel_link">
+    <gazebo reference="${robot_prefix}/left_wheel_link">
         <material>Gazebo/Grey</material>
     </gazebo>
-    <gazebo reference="caster_wheel_link">
+    <gazebo reference="${robot_prefix}/caster_wheel_link">
         <material>Gazebo/Grey</material>
         <mu1 value="0.1" />
@@ -223,6 +212,6 @@
             <update_rate>50</update_rate>
             <!-- wheels -->
-            <left_joint>base_left_wheel_joint</left_joint>
-            <right_joint>base_right_wheel_joint</right_joint>
+            <left_joint> ${robot_prefix}/base_left_wheel_joint </left_joint>
+            <right_joint> ${robot_prefix}/base_right_wheel_joint </right_joint>
             <!-- kinematics -->
             <wheel_separation>0.45</wheel_separation>
@@ -232,7 +221,7 @@
             <publish_odom_tf>true</publish_odom_tf>
             <publish_wheel_tf>true</publish_wheel_tf>
-            <odometry_topic>odom</odometry_topic>
-            <odometry_frame>odom</odometry_frame>
-            <robot_base_frame>base_footprint</robot_base_frame>
+            <odometry_topic>${robot_prefix}/odom</odometry_topic>
+            <odometry_frame>${robot_prefix}/odom</odometry_frame>
+            <robot_base_frame> ${robot_prefix}/base_footprint </robot_base_frame>
         </plugin>
     </gazebo>

Commit message: Launch multiple robots lidar

File: src/OfficeEnv/urdf/my_robot.urdf.xacro (robot description, xacro)
@@ -226,3 +226,58 @@
         </plugin>
     </gazebo>
+    <joint name="${robot_prefix}/laser_joint" type="fixed">
+        <parent link="${robot_prefix}/base_link"/>
+        <child link="${robot_prefix}/laser_frame"/>
+        <origin xyz="0.122 0 0.212" rpy="0 0 0"/>
+    </joint>
+    <link name="${robot_prefix}/laser_frame">
+        <visual>
+            <geometry>
+                <cylinder radius="0.05" length="0.04"/>
+            </geometry>
+            <material name="grey"/>
+        </visual>
+        <visual>
+            <origin xyz="0 0 -0.05"/>
+            <geometry>
+                <cylinder radius="0.01" length="0.1"/>
+            </geometry>
+            <material name="grey"/>
+        </visual>
+        <collision>
+            <geometry>
+                <cylinder radius="0.05" length="0.04"/>
+            </geometry>
+        </collision>
+        <xacro:cylinder_inertia m="0.1" r="0.05" h="0.04"
+                                    xyz="0 0 0" rpy="0 0 0" />
+    </link>
+    <gazebo reference="${robot_prefix}/laser_frame">
+        <material>Gazebo/grey</material>
+        <sensor name="${robot_prefix}/laser" type="ray">
+            <pose> 0 0 0 0 0 0 </pose>
+            <visualize>true</visualize>
+            <update_rate>10</update_rate>
+            <ray>
+                <scan>
+                    <horizontal>
+                        <samples>360</samples>
+                        <min_angle>-3.14</min_angle>
+                        <max_angle>3.14</max_angle>
+                    </horizontal>
+                </scan>
+                <range>
+                    <min>0.3</min>
+                    <max>12</max>
+                </range>
+            </ray>
+            <plugin name="laser_controller" filename="libgazebo_ros_ray_sensor.so">
+                <ros>
+                    <argument>~/out:=scan</argument>
+                </ros>
+                <output_type>sensor_msgs/LaserScan</output_type>
+                <frame_name>${robot_prefix}/laser_frame</frame_name>
+            </plugin>
+        </sensor>
+    </gazebo>
 </robot>
